File: FC_Remote-hardware/Battery.kicad_sch (KiCad schematic)
At the start: 19 parts, among them U3 BQ25185DLHR

Commit message: added changes
Parts:
- removed C13: 100uF, Capacitor_THT:C_Radial_D6.3mm_H5.0mm_P2.50mm, symbol Device:C
- removed C16: 10uF, Capacitor_SMD:C_0603_1608Metric, symbol Device:C
- removed C17: 0.1uF, Capacitor_SMD:C_0603_1608Metric, symbol Device:C
- removed R22, R23: 100K, Resistor_SMD:R_0603_1608Metric, symbol Device:R
- removed R7: 10K, Resistor_SMD:R_0603_1608Metric, symbol Device:R
- added C3: 1uF, Capacitor_SMD:C_0603_1608Metric, symbol Device:C
- added R27, R28: 10K, Resistor_SMD:R_0603_1608Metric, symbol Device:R
- R12: value 18K -> 13K
- R2, R6: value 1K -> 5K
Connections:
- net +5V: now also C3.1
- net GND: now also BT1.1 (+), U3.4 (~{CE}), C3.2, R28.1; no longer BT1.2 (-)
- net VBAT: now also BT1.2 (-), R27.1; no longer BT1.1 (+)
- new net BATT_ADC: R27.2, R28.2
Other:
- note added: "For the battery we use this needs to happen lol"
- moved on the sheet: BT1, C2, C4, D3, D4, D6, R12, R13, R14, R15, R2, R6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
