File: FC_Remote-hardware/ESP32.kicad_sch (KiCad schematic)
At the start: 14 parts, among them Q3 MMBT2222A, Q4 MMBT2222A, SW1 SW_Push, SW4 SW_Push, U6 ESP32-WROOM-32D, U9 CH340C

Commit message: added changes
Parts:
- removed C3: 1uF, Capacitor_SMD:C_0603_1608Metric, symbol Device:C
- removed U6: ESP32-WROOM-32D, RF_Module:ESP32-WROOM-32D, symbol RF_Module:ESP32-WROOM-32D
- added C10, C12, C9: 1uF, Capacitor_SMD:C_0603_1608Metric, symbol Device:C
- added C11: 10uF, Capacitor_SMD:C_0603_1608Metric, symbol Device:C
- added C15, C16, C17, C18, C19, C20: 0.1uF, Capacitor_SMD:C_0603_1608Metric, symbol Device:C
- added R1, R5: 10k, Resistor_SMD:R_0603_1608Metric, symbol Device:R
- added R19: 10K, Resistor_SMD:R_0603_1608Metric, symbol Device:R
- added U5: ESP32-WROVER-E-N16R8, PCM_SparkFun-RF:ESP32-WROVER-E-IE, symbol PCM_SparkFun-RF:ESP32-WROVER-E-N16R8
- R20, R21: value R -> 470
- R8: value 10k -> 10K
Connections:
- net +3.3V: now also C10.1, C11.2, C12.2, C19.2, C20.2, R1.2, R5.1, U5.2 (VDD); no longer R8.1
- net 0_ESP: now also R1.1, U5.25 (IOA0)
- net CHIP_PU: now also C9.1, R5.2, U5.3 (EN); no longer R8.2
- net GND: now also R8.2, U9.15 (R232), C10.2, C11.1, C12.1, C15.2, C16.2, C17.2, C18.2, C19.1, C20.1, C9.2, R19.2, U5.1 (GND), U5.15 (GND), U5.38 (GND), U5.39.1 (GND), U5.39.2 (GND), U5.39.3 (GND), U5.39.4 (GND), U5.39.5 (GND), U5.39.6 (GND), U5.39.7 (GND), U5.39.8 (GND), U5.39.9 (GND)
- net RX_ESP: now also U5.34 (RXD0/IO3)
- net TX_ESP: now also U5.35 (TXD0/IO1)
- new net AUTONOMY_SW: R8.1, U5.5 (IA39)
- new net BATT_ADC: C15.1, U5.9 (IOA33)
- new net CTRL_CE: U5.31 (IO19)
- new net CTRL_CSN: U5.24 (IOA2)
- new net CTRL_IRQ: U5.14 (IOA12)
- new net DIR_JOY_BTN: U5.23 (IOA15)
- new net DIR_JOY_X: C16.1, U5.7 (IA35)
- new net DIR_JOY_Y: C18.1, U5.8 (IOA32)
- new net FLIGHT_MODE_SW: R19.1, U5.4 (IA36)
- new net NRF_MISO: U5.12 (IOA27)
- new net NRF_MOSI: U5.16 (IOA13)
- new net NRF_SCK: U5.13 (IOA14)
- new net TELM_CE: U5.26 (IOA4)
- new net TELM_CSN: U5.29 (IO5)
- new net TELM_IRQ: U5.11 (IOA26)
- new net TFT_BL: U5.10 (IOA25)
- new net TFT_CS: U5.33 (IO21)
- new net TFT_DC: U5.36 (IO22)
- new net TFT_MOSI: U5.37 (IO23)
- new net TFT_SCK: U5.30 (IO18)
- new net THROTTLE_JOY: C17.1, U5.6 (IA34)
- no-connect marks 15 -> 4
Other:
- note added: "GPIO 0 (must be LOW to enter boot mode)"
- note added: "GPIO 12 (must be LOW on boot)"
- note added: "GPIO 15 (must be HIGH during boot)"
- note added: "GPIO 2 (must be floating or LOW during boot)"
- note added: "GPIO 5 (must be HIGH during boot)"
- note added: "IA34-39 - no internal pull-ups, need external ones if used as inputs"
- note added: "Place these close to the modueles supply"
- note added: "wanted smoother ADC readings"
- note removed: "ADC1_CH0 (GPIO 36) ADC1_CH1 (GPIO 37) ADC1_CH2 (GPIO 38) ADC1_CH3 (GPIO 39) ADC1_CH4 (GPIO 32) ADC1_CH5 (GPIO 33) ADC1_CH6 (GPIO 34) ADC1_CH7 (GPIO 35) ADC2_CH0 (GPIO 4) ADC2_CH1 (GPIO 0) ADC2_CH2 (GPIO 2) ADC2_CH3 (GPIO 15) ADC2_CH4 (GPIO 13) ADC2_CH5 (GPIO 12) ADC2_CH6 (GPIO 14) ADC2_CH7 (GPIO 27) ADC2_CH8 (GPIO 25) ADC2_CH9 (GPIO 26)"
- note removed: "Strapping Pins The ESP32 chip has the following strapping pins: GPIO 0 (must be LOW to enter boot mode) GPIO 2 (must be floating or LOW during boot) GPIO 4 GPIO 5 (must be HIGH during boot) GPIO 12 (must be LOW during boot) GPIO 15 (must be HIGH during boot)"
- moved on the sheet: D1, D2, Q3, Q4, R10, R20, R21, R9, SW1, SW4, U9
