File: FC_Remote-hardware/SPI.kicad_sch (KiCad schematic)
At the start: 14 parts, among them SW3 SW_Push, SW6 SW_Push, U1 COM-09032, U12 NRF24L01_Breakout, U2 COM-09032, U4 ST7789_2IN_WS, U7 NRF24L01_Breakout

Commit message: added changes
Parts:
- removed BZ1: Buzzer, Buzzer_Beeper:Buzzer_12x9.5RM7.6, symbol Device:Buzzer
- removed R1: DNP, Resistor_SMD:R_0603_1608Metric, symbol Device:R
- removed SW3, SW6: SW_Push, Button_Switch_SMD:SW_Push_1P1T_NO_CK_PTS125Sx85SMTR, symbol Switch:SW_Push
- added C13: 1uF, Capacitor_SMD:C_0603_1608Metric, symbol Device:C
- added C14: 0.1uF, Capacitor_SMD:C_0603_1608Metric, symbol Device:C
- added C21, C22: 22uF, PCM_SparkFun-Capacitor:C_0805_2012Metric, symbol PCM_SparkFun-Capacitor:22uF_0805_25V_20%
- added D10, D8: GREEN, LED_SMD:LED_0603_1608Metric_Pad1.05x0.95mm_HandSolder, symbol Device:LED
- added R7: 5K, Resistor_SMD:R_0603_1608Metric_Pad0.98x0.95mm_HandSolder, symbol Device:R
- added SW2, SW3: SW_SPST, SWITCHMTS101:mts101sw, symbol Switch:SW_SPST
- R11: value DNP -> 5K; footprint Resistor_SMD:R_0603_1608Metric -> Resistor_SMD:R_0603_1608Metric_Pad0.98x0.95mm_HandSolder
Connections:
- net I34_ESP is gone; now on net GND: U1.H2 (H)
- net SAMD_MISO is gone; now on net NRF_MISO: U7.7 (MISO)
- net SAMD_MOSI is gone; now on net NRF_MOSI: U7.6 (MOSI)
- net +3.3V: now also C13.1, C14.1, C21.1, C22.1, R7.1, SW2.2 (B), SW3.2 (B); no longer U1.H1 (H+)
- net GND: now also U1.B1A (SEL+), U1.H1 (H+), C13.2, C14.2, C21.2, C22.2, D10.1 (K), D8.1 (K)
- net TELM_IRQ: now reaches U7.8 (IRQ)
- net DIR_JOY_BTN: now reaches U2.B1A (SEL+)
- net CTRL_IRQ: now reaches U12.8 (IRQ)
- net 14_ESP renamed DIR_JOY_X
- net 17_ESP renamed TFT_CS
- net 21_ESP renamed CTRL_CSN
- net 27_ESP renamed TFT_DC
- net 32_ESP renamed CHIP_PU
- net 33_ESP renamed TFT_BL
- net A1_ESP renamed CTRL_CE
- net A5_ESP renamed DIR_JOY_Y
- net I35_ESP renamed THROTTLE_JOY
- net MISO_ESP renamed NRF_MISO
- net MOSI_ESP renamed NRF_MOSI
- net NRF_MOSI: no longer U4.3 (DIN)
- net SAMD_A0 renamed TELM_CSN
- net SAMD_A1 renamed TELM_CE
- net SAMD_SCK renamed NRF_SCK
- net NRF_SCK: now also U12.5 (SCK)
- net SAMD_SCL: no longer names the net of R11.2
- net SAMD_SCL: now also D10.2 (A)
- net SCK_ESP renamed TFT_SCK
- net TFT_SCK: no longer U12.5 (SCK)
- new net: D8.2 (A), R7.2
- new net AUTONOMY_SW: SW3.1 (A)
- new net FLIGHT_MODE_SW: SW2.1 (A)
- new net TFT_MOSI: U4.3 (DIN)
- no-connect marks 4 -> 0
Other:
- moved on the sheet: U1, U2
