File: FC_Remote-hardware/power_for_remote.kicad_sch (KiCad schematic)
At the start: 22 parts, among them J1 USB_C_Receptacle, J2 USB_C_Receptacle, SW8 SW_SPST, U8 TPS63802DLAR

Commit message: added changes
Parts:
- removed C19: 10uF, Capacitor_SMD:C_0603_1608Metric, symbol Device:C
- removed C20: 0.1uF, Capacitor_SMD:C_0603_1608Metric, symbol Device:C
- removed D7, D8: PESD0603-240, PCM_SparkFun-Capacitor:C_0603_1608Metric, symbol PCM_SparkFun-DiscreteSemi:D_TVS_0603_24V
- removed F1, F2: Polyfuse, Fuse:Fuse_1206_3216Metric, symbol Device:Polyfuse
- removed J2: USB_C_Receptacle, PCM_SparkFun-Connector:USB-C_16, symbol PCM_SparkFun-Connector:USB_C_Receptacle
- removed R19, R5: 5.1k, Resistor_SMD:R_0603_1608Metric, symbol Device:R
- removed R24: 100K, Resistor_SMD:R_0603_1608Metric_Pad0.98x0.95mm_HandSolder, symbol Device:R
- added D7: PMEG4020EJ, Diode_SMD:D_SOD-323, symbol Device:D_Schottky
- added U6: TPD2EUSB30, Package_TO_SOT_SMD:Texas_DRT-3, symbol Power_Protection:TPD2EUSB30
- R3: value 500 -> 5K
Connections:
- net +5V: now also D7.1 (K)
- net GND: now also U6.3 (GND)
- net USB_D+_ESP: now also U6.1 (D+)
- net USB__D-_ESP: now also U6.2 (D-)
- net at J1.VBUS: now also D7.2 (A)
- no-connect marks 0 -> 1
Other:
- note added: "Place this as close as possible"
- moved on the sheet: C1, C5, D5, L1, R16, R17, R3, SW8, U8
